File: stepper-motor-controller.kicad_pcb (KiCad board)
At the start: 2 copper layers, 39 parts, among them U5 TMC5160A-TA-T

Commit message: b
Parts:
- added J1: Conn_01x07, Connector_PinHeader_2.54mm:PinHeader_1x07_P2.54mm_Vertical, F.Cu at (119.4, 59.4)
- added J2: Conn_01x03, Connector_PinHeader_2.54mm:PinHeader_1x03_P2.54mm_Vertical, F.Cu at (126.5, 52.3)
- added J3: Conn_01x04, Connector_PinHeader_2.54mm:PinHeader_1x04_P2.54mm_Vertical, F.Cu at (169.2, 61.5)
- C2: footprint Capacitor_SMD:C_0603_1608Metric_Pad1.08x0.95mm_HandSolder -> Capacitor_SMD:C_0805_2012Metric_Pad1.18x1.45mm_HandSolder
- R1, R10, R14, R15, R2, R7, R8, R9: footprint Resistor_SMD:R_0603_1608Metric_Pad0.98x0.95mm_HandSolder -> Resistor_SMD:R_2512_6332Metric_Pad1.40x3.35mm_HandSolder
- U1, U2, U3, U4, U6, U7, U8, U9: value ~ -> AOD4126
- moved R10 118.4 mm to (119.4, 82.3), turned to -90 degrees
- moved R14 112.9 mm to (127.0, 86.9), turned to 90 degrees
- moved C3 103.1 mm to (140.0, 51.6), turned to 0 degrees
- moved R13 97.6 mm to (141.0, 90.4)
- moved R11 96.7 mm to (141.0, 88.4)
- moved R12 96.2 mm to (141.0, 92.5)
- moved R1 92.9 mm to (137.2, 47.2)
- moved R15 92.4 mm to (149.4, 88.9), turned to 180 degrees
- moved U2 88.1 mm to (147.4, 51.6), turned to 180 degrees
- moved R4 85.0 mm to (144.5, 64.8)
- moved R5 84.7 mm to (144.5, 68.8)
- moved R6 84.6 mm to (144.5, 66.8)
- moved R2 84.3 mm to (129.0, 47.2)
- moved U9 81.3 mm to (144.0, 83.3), turned to 180 degrees
- moved C13 81.0 mm to (136.5, 75.2)
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Connections:
- net /12VOUT renamed /TMC5160A/12VOUT
- net /5VOUT renamed /TMC5160A/5VOUT
- net /CPI renamed /TMC5160A/CPI
- net /CPO renamed /TMC5160A/CPO
- net /VCC renamed /TMC5160A/VCC
- net /VCP renamed /TMC5160A/VCP
- C12 pad 1: /BMA2 -> /BMB2
- C12 pad 2: /CA2 -> /CB2
- C13 pad 1: /CB1 -> /CA1
- C13 pad 2: /BMB1 -> /BMA1
- C15 pad 1: /BMB2 -> /BMA2
- C15 pad 2: /CB2 -> /CA2
- C3 pad 1: /CA1 -> /CB1
- C3 pad 2: /BMA1 -> /BMB1
- R1 pad 1: /HA1 -> /HB1
- R10 pad 1: /LB1 -> /LA1
- R11 pad 1: /SRBH -> /SRAH
- R12 pad 1: /SRBL -> /SRAL
- R14 pad 2: /HB2 -> /HA2
- R15 pad 2: /LB2 -> /LA2
- R2 pad 1: /LA1 -> /LB1
- R4 pad 1: /SRAH -> /SRBH
- R5 pad 1: /SRAL -> /SRBL
- R7 pad 2: /HA2 -> /HB2
- R8 pad 2: /LA2 -> /LB2
- R9 pad 1: /HB1 -> /HA1
- U1 pad 3: /BMA1 -> /BMB1
- U2 pad 2: /BMA1 -> /BMB1
- U3 pad 3: /BMA2 -> /BMB2
- U4 pad 2: /BMA2 -> /BMB2
- U5 pad 13: /CSN -> /TMC5160A/CSN
- U5 pad 14: /SCK -> /TMC5160A/SCK
- U5 pad 15: /MOSI -> /TMC5160A/MOSI
- U5 pad 16: /MISO -> /TMC5160A/MISO
- U5 pad 26: /DIAG0 -> /TMC5160A/DIAG0
- U5 pad 27: /DIAG1 -> /TMC5160A/DIAG1
- U5 pad 28: /ENABLE -> /TMC5160A/ENABLE
- U6 pad 3: /BMB1 -> /BMA1
- U7 pad 2: /BMB1 -> /BMA1
- U8 pad 3: /BMB2 -> /BMA2
- U9 pad 2: /BMB2 -> /BMA2
Routing:
- net /BMB1: track 0.00 -> 95.4 mm, vias 0 -> 1
- net VM: track 60.8 -> 149.8 mm, vias 2 -> 4
- net /BMB2: track 0.00 -> 77.3 mm, vias 0 -> 3
- net Net-(U2-S): track 11.5 -> 66.1 mm, vias 0 -> 6
- net /HB2: track 0.00 -> 46.6 mm, vias 0 -> 2
- net /SRBL: track 0.00 -> 43.5 mm, vias 0 -> 6
- net /SRAH: track 0.00 -> 42.7 mm, vias 0 -> 2
- net /BMA1: track 13.1 -> 53.5 mm, vias 0 -> 1
- net /SRBH: track 0.00 -> 38.8 mm, vias 0 -> 4
- net /SRAL: track 0.00 -> 37.0 mm, vias 0 -> 2
- net /BMA2: track 18.6 -> 55.0 mm, vias 0 -> 1
- net Net-(U8-G): track 0.00 -> 34.5 mm, vias 0 -> 2
- net Net-(U7-G): track 0.00 -> 32.5 mm, vias 0 -> 2
- net /LA1: track 0.00 -> 29.0 mm, vias 0 -> 2
- net GND: track 48.2 -> 74.5 mm, vias 0 -> 33
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- added copper zone on B.Cu, net GND
Other:
- board outline added: 54.4 x 49.3 mm
