File: stepper-motor-controller.kicad_sch (KiCad schematic)
At the start: 39 parts, among them U5 TMC5160A-TA-T

Commit message: b
Parts:
- removed C1, C10: 100nF, Capacitor_SMD:C_0603_1608Metric_Pad1.08x0.95mm_HandSolder, symbol Device:C
- removed C11, C2, C4, C5, C7, C9: 2.2uF, Capacitor_SMD:C_0603_1608Metric_Pad1.08x0.95mm_HandSolder, symbol Device:C
- removed C12, C13, C14, C15, C3, C6, C8: 470nF, Capacitor_SMD:C_0603_1608Metric_Pad1.08x0.95mm_HandSolder, symbol Device:C
- removed R1, R10, R14, R15, R2, R7, R8, R9: 5, Resistor_SMD:R_0603_1608Metric_Pad0.98x0.95mm_HandSolder, symbol Device:R
- removed R11, R12, R4, R5: 47, Resistor_SMD:R_0603_1608Metric_Pad0.98x0.95mm_HandSolder, symbol Device:R
- removed R13, R6: 30m, Resistor_SMD:R_0603_1608Metric_Pad0.98x0.95mm_HandSolder, symbol Device:R
- removed R3: 2.2, Resistor_SMD:R_0603_1608Metric_Pad0.98x0.95mm_HandSolder, symbol Device:R
- removed U1, U2, U3, U4, U6, U7, U8, U9: ~, AOD4126:TRANS_TSM60N1R4CP_ROG, symbol AOD4126:AOD4126
- removed U5: TMC5160A-TA-T, TMC5160A-TA-T:21-100582_ADI, symbol 2025-02-07_15-41-28:TMC5160A-TA-T
- added J1: Conn_01x07, Connector_PinHeader_2.54mm:PinHeader_1x07_P2.54mm_Vertical, symbol Connector_Generic:Conn_01x07
- added J2: Conn_01x03, Connector_PinHeader_2.54mm:PinHeader_1x03_P2.54mm_Vertical, symbol Connector_Generic:Conn_01x03
- added J3: Conn_01x04, Connector_PinHeader_2.54mm:PinHeader_1x04_P2.54mm_Vertical, symbol Connector_Generic:Conn_01x04
Connections:
- net GND: now also J2.1 (Pin_1)
- net VC: now also J2.3 (Pin_3)
- net VM: now also J2.2 (Pin_2)
- new net HBridge1/M1: J3.1 (Pin_1)
- new net HBridge1/M2: J3.2 (Pin_2)
- new net HBridge2/M1: J3.3 (Pin_3)
- new net HBridge2/M2: J3.4 (Pin_4)
- new net TMC5160A/CSN: J1.1 (Pin_1)
- new net TMC5160A/DIAG0: J1.6 (Pin_6)
- new net TMC5160A/DIAG1: J1.7 (Pin_7)
- new net TMC5160A/ENABLE: J1.5 (Pin_5)
- new net TMC5160A/MISO: J1.4 (Pin_4)
- new net TMC5160A/MOSI: J1.3 (Pin_3)
- new net TMC5160A/SCK: J1.2 (Pin_2)
Other:
- added sheet HBridge1 (hbridge.kicad_sch)
- added sheet HBridge2 (hbridge.kicad_sch)
- added sheet TMC5160A (TMC5160A.kicad_sch)
